Commit message: increase elbow joint range
new range: [0,150]
rad: [0,2.617993878]

File: arm_1dof/demo_human_col/skeleton.urdf (robot description, URDF)
Before this commit: robot skeleton, 10 links, 9 joints
Joints:
- joint skeleton__elbow_joint: limit lower=0.0 upper=1.5707963705062866 effort=0.0 velocity=0.0 -> lower=0.0 upper=2.617993878 effort=0.0 velocity=0.0

Commit message: feat: make shoulder revolute joint

File: arm_1dof/demo_human_col/skeleton.urdf (robot description, URDF)
Before this commit: robot skeleton, 10 links, 9 joints
Joints:
- joint skeleton__shoulder_joint: axis 0 0 1 -> 1 0 0; limit lower=-0.1 upper=0.7853981852531433 effort=0.0 velocity=0.0 -> lower=-1 upper=0.7853981852531433 effort=0.0 velocity=0.0; type fixed -> revolute

Commit message: feat: allow knuckle joint to rotate

File: arm_1dof/demo_human_col/skeleton.urdf (robot description, URDF)
Before this commit: robot skeleton, 10 links, 9 joints
Joints:
- joint skeleton__proximal_joint: type fixed -> revolute
